Commit message: Passage à la nouvelle version
Obligé de changer tout les documents puisque le répertoire de Franka a changé de version. Cette version permet de faire bouger le robot. Elle incorpore aussi des changements dans certains programmes notamment dans le dossier controller.

File: franka_fr3_moveit_config/srdf/fr3_arm.srdf.xacro (robot description, xacro)
@@ -5,5 +5,5 @@
   <xacro:property name="arm_id" value="$(arg arm_id)"/>
   <xacro:include filename="$(find franka_fr3_moveit_config)/srdf/fr3_arm.xacro"/>
-  <xacro:fr3_arm arm_id="${arm_id}"/>
+  <xacro:fr3_arm arm_id="${arm_id}" hand="$(arg hand)"/>
   <xacro:if value="$(arg hand)">
     <xacro:include filename="$(find franka_fr3_moveit_config)/srdf/hand.xacro"/>

File: franka_fr3_moveit_config/srdf/fr3_arm.xacro (robot description, xacro)
@@ -1,7 +1,9 @@
 <?xml version="1.0" ?>
 <robot xmlns:xacro="http://www.ros.org/wiki/xacro" name="fr3">
-  <xacro:macro name="fr3_arm" params="arm_id:='fr3' ">
+  <xacro:macro name="fr3_arm" params="arm_id:='fr3' hand:='true' ">
     <xacro:include filename="$(find franka_fr3_moveit_config)/srdf/group_definition.xacro"/>
-    <xacro:group_definition arm_id="${arm_id}" group_name="${arm_id}_manipulator" tip_link="${arm_id}_hand_tcp"/>
+    <xacro:if value="${hand}">
+      <xacro:group_definition arm_id="${arm_id}" group_name="${arm_id}_manipulator" tip_link="${arm_id}_hand_tcp"/>
+    </xacro:if>
     <xacro:group_definition arm_id="${arm_id}" group_name="${arm_id}_arm" tip_link="${arm_id}_link8"/>
     <virtual_joint name="virtual_joint" type="fixed" parent_frame="world" child_link="${arm_id}_link0"/>
